File: Unicycle Battery.kicad_pcb (KiCad board)
At the start: 2 copper layers, 230 x 290 mm, 0 parts

Commit message: PCB Guestimate complete (tm)
Parts:
- added BT1: ~, Unicycle:P Group, F.Cu at (74.0, 176.6)
- added BT10: ~, Unicycle:P Group, F.Cu at (73.0, 110.8)
- added BT11: ~, Unicycle:P Group, F.Cu at (146.0, 109.8)
- added BT12: ~, Unicycle:P Group, F.Cu at (215.0, 109.8)
- added BT2: ~, Unicycle:P Group, F.Cu at (74.0, 242.2)
- added BT3: ~, Unicycle:P Group, F.Cu at (74.0, 307.8)
- added BT4: ~, Unicycle:P Group, F.Cu at (148.1, 176.6)
- added BT5: ~, Unicycle:P Group, F.Cu at (148.1, 242.2)
- added BT6: ~, Unicycle:P Group, F.Cu at (148.1, 307.8)
- added BT7: ~, Unicycle:P Group, F.Cu at (222.1, 176.6)
- added BT8: ~, Unicycle:P Group, F.Cu at (222.1, 242.2)
- added BT9: ~, Unicycle:P Group, F.Cu at (222.1, 307.8)

Commit message: First draft
Done:
One pad per connection
Alignment done
All components added

TODO:
Via stitching
Clean up traces + increase width
Remove or stitch top layer pads
Double check math
Parts:
- added J1: S13B-PH-K-S, Connector_JST:JST_PH_S13B-PH-K_1x13_P2.00mm_Horizontal, F.Cu at (159.2, 60.2)
- added J2: XT60PW-F, Connector_AMASS:AMASS_XT60PW-F_1x02_P7.20mm_Horizontal, F.Cu at (239.3, 69.0)
- added J3: XT30PW-F, Connector_AMASS:AMASS_XT30PW-F_1x02_P2.50mm_Horizontal, F.Cu at (204.0, 68.2)
- BT1, BT2, BT7, BT8: footprint Unicycle:P Group -> Unicycle:P Group Even
- BT10, BT3, BT4, BT9: footprint Unicycle:P Group -> Unicycle:P Group End
- BT11, BT5: footprint Unicycle:P Group -> Unicycle:P Group 4-5 10-11
- BT12, BT6: footprint Unicycle:P Group -> Unicycle:P Group 5-6 11-+
- moved BT9 199.8 mm to (75.0, 172.6)
- moved BT1 195.0 mm to (219.0, 307.1)
- moved BT8 102.4 mm to (147.0, 172.6)
- moved BT6 98.3 mm to (219.0, 239.8), turned to 180 degrees
- moved BT2 97.6 mm to (147.0, 307.1)
- moved BT4 96.6 mm to (75.0, 239.8), turned to 180 degrees
- moved BT12 6.02 mm to (219.0, 105.3), turned to 180 degrees
- moved BT10 5.85 mm to (75.0, 105.3), turned to 180 degrees
- moved BT7 5.10 mm to (219.0, 172.6)
- moved BT11 4.61 mm to (147.0, 105.3), turned to 180 degrees
- moved BT5 2.62 mm to (147.0, 239.8), turned to 180 degrees
- moved BT3 1.25 mm to (75.0, 307.1)
Connections:
- net Net-(BT10-Pad-) renamed /9
- net Net-(BT3-Pad+) renamed /3
- net Net-(BT6-Pad+) renamed /6
- BT10 pad +: Net-(BT10-Pad+) -> /10
- BT11 pad +: Net-(BT11-Pad+) -> /11
- BT2 pad -: Net-(BT1-Pad+) -> /1
- BT3 pad -: Net-(BT2-Pad+) -> /2
- BT4 pad +: Net-(BT4-Pad+) -> /4
- BT5 pad +: Net-(BT5-Pad+) -> /5
- BT8 pad -: Net-(BT7-Pad+) -> /7
- BT9 pad -: Net-(BT8-Pad+) -> /8
Routing:
- net /2: track 0.00 -> 269.7 mm, vias 0 -> 2
- net /1: track 0.00 -> 252.9 mm, vias 0 -> 2
- net /3: track 0.00 -> 248.5 mm, vias 0 -> 1
- net /6: track 0.00 -> 227.9 mm
- net /4: track 0.00 -> 213.7 mm, vias 0 -> 1
- net /5: track 0.00 -> 189.0 mm, vias 0 -> 1
- net /8: track 0.00 -> 182.3 mm, vias 0 -> 1
- net +BATT: track 0.00 -> 149.7 mm, vias 0 -> 1
- net /7: track 0.00 -> 124.7 mm
- net /9: track 0.00 -> 112.5 mm, vias 0 -> 136
- net /11: track 0.00 -> 59.4 mm
- net /10: track 0.00 -> 52.2 mm
- net -BATT: track 0.00 -> 50.1 mm
- added copper zone on B.Cu, net -BATT
- added copper zone on F.Cu, net -BATT
- added copper zone on B.Cu, net /3
- added copper zone on F.Cu, net /3
- added copper zone on B.Cu, net /6
- added copper zone on F.Cu, net /6
- added copper zone on B.Cu, net /9
- added copper zone on F.Cu, net /9
Other:
- board text added: "TODO: Via stitching Clean up traces + increase width Remove or stitch top layer pads Double check math"

Commit message: Finished PCB
Parts:
- added H1: MountingHole, MountingHole:MountingHole_4.3mm_M4, F.Cu at (38.0, 57.0)
- added H2: MountingHole, MountingHole:MountingHole_4.3mm_M4, F.Cu at (256.0, 57.0)
Routing:
- net /9: track 112.5 -> 75.0 mm, vias 136 -> 141
- net /10: track 52.2 -> 67.6 mm, vias 0 -> 1
- net -BATT: track 50.1 -> 65.2 mm, vias 0 -> 137
- net /8: vias 1 -> 2
- net /7: vias 0 -> 1
- net /6: vias 0 -> 108
- net /5: vias 1 -> 2
- net /4: vias 1 -> 2
- net /3: vias 1 -> 142
- net /2: vias 2 -> 3
- net /11: vias 0 -> 1
- net /1: vias 2 -> 3
- net +BATT: vias 1 -> 2
- added copper zone on F.Cu, net +BATT
Other:
- outline, holes or cut-outs redrawn
- board text removed: "TODO: Via stitching Clean up traces + increase width Remove or stitch top layer pads Double check math"
